File: lora-module.kicad_pcb (KiCad board)
At the start: 4 copper layers, 20.3 x 21.7 mm, 53 parts, among them J101 Conn_Coaxial, J102 Conn_ARM_SWD_TagConnect_TC203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, Q101 PMN48XP, U201 STM32WLE5CCUx, U301 BALFHB-WL-05D3, U302 BGS12SN6E6327XTSA1, U401 SST26VF080A

Commit message: added teardrops, finishing touches
Routing:
- net GND: track 26.1 -> 27.7 mm, vias 59 -> 73
Other:
- board size 20.3 x 21.7 mm -> 20.3 x 22.5 mm
